Commit message: Tweaks for getting Lab 1 working

File: lynx/al5d_description/urdf/al5d.xacro (robot description, xacro)
@@ -3,8 +3,8 @@
     <xacro:include filename="$(find al5d_description)/urdf/transmissions.urdf.xacro"/>
     <xacro:property name="M_PI" value="3.14159"/>
-    <xacro:property name="base_height" value="0.43" />
+    <xacro:property name="base_height" value="0.02" />
     <xacro:property name="base_radius" value="0.048" />
-    <xacro:property name="upper_base_height" value="0.006" />
-    <xacro:property name="upper_arm_offset" value="0.022" />
+    <xacro:property name="upper_base_height" value="0.07" />
+    <xacro:property name="upper_arm_offset" value="0.006" />
     <xacro:property name="upper_arm_length" value="0.14605" />
     <xacro:property name="upper_arm_width" value="0.05" />
@@ -45,7 +45,7 @@
     <link name="upper_base">
       <visual>
-        <origin xyz="0 0 0" rpy="0 0 0"/>
-        <geometry>
-          <cylinder length="${upper_base_height}" radius="${base_radius}"/>
+	<origin xyz="0 0 ${(upper_base_height - base_height - 0.02)/2 + base_height + 0.02}" rpy="0 0 0"/>
+        <geometry>
+          <cylinder length="${upper_base_height - base_height - 0.02}" radius="${base_radius}"/>
         </geometry>
         <material name="black">
@@ -53,7 +53,7 @@
       </visual>
       <collision>
-        <origin xyz="0 0 0" rpy="0 0 0"/>
-        <geometry>
-           <cylinder length="${upper_base_height}" radius="${base_radius}"/>
+	<origin xyz="0 0 ${(upper_base_height - base_height - 0.02)/2 + base_height + 0.02}" rpy="0 0 0"/>
+        <geometry>
+          <cylinder length="${upper_base_height - base_height - 0.02}" radius="${base_radius}"/>
         </geometry>
       </collision>
@@ -176,5 +176,5 @@
     </joint>
     <joint name="base_rotate" type="revolute">
-      <origin xyz="0 0 ${base_height + upper_base_height}" rpy="0 0 0"/>
+      <origin xyz="0 0 0" rpy="0 0 0"/>
       <parent link="base"/>
       <child link="upper_base"/>
@@ -183,5 +183,5 @@
     </joint>
     <joint name="shoulder_tilt" type="revolute">
-      <origin xyz="0 0 ${upper_arm_offset}" rpy="${M_PI/2} -${M_PI/2} 0 "/>
+      <origin xyz="0 0 ${upper_arm_offset + upper_base_height}" rpy="${M_PI/2} -${M_PI/2} 0 "/>
       <parent link="upper_base"/>
       <child link="upper_arm"/>
@@ -225,5 +225,5 @@
     </joint>
     <joint name="end" type="fixed">
-      <origin xyz="${wrist_length} 0 0" rpy="0 0 0"/>
+      <origin xyz="${wrist_length} 0 0" rpy="0 ${M_PI/2} 0"/>
       <parent link="gripper_base"/>
       <child link="end"/>
