Commit message: update lidar joint and controller

File: al5d_description/urdf/al5d_lidar (copy).xacro (robot description, xacro)
@@ -16,4 +16,5 @@
     <xacro:property name="gripper_width" value="0.05" />
     <xacro:property name="gripper_height" value="0.01" />
+    <xacro:property name="finger_length" value="0.04" />
     <xacro:property name="inertia_block">
       <inertial>
@@ -130,29 +131,4 @@
       <xacro:insert_block name="inertia_block" />
     </link>
-    <link name="lidar">
-      <visual>
-	<origin xyz="0 0 0" rpy="0 0 0"/>
-        <geometry>
-          <box size="0.0212 0.0522 0.024"/>
-        </geometry>
-        <material name="red">
-          <color rgba="1 0.3 0.3 0.85"/>
-        </material>
-      </visual>
-      <collision>
-        <origin xyz="0 0 0" rpy="0 0 0"/>
-        <geometry>
-          <box size="0.0212 0.0522 0.024"/>
-        </geometry>
-      </collision>
-      <xacro:insert_block name="inertia_block" />
-    </link>
-  <joint name="lidar_rotate" type="revolute">
-    <origin xyz="0 0 -0.035" rpy="0 0 0" />
-    <parent link="gripper_base"/>
-    <child link="lidar" />
-    <axis xyz="0 0 1"/>
-    <limit lower="-1.4" upper="1.4" effort="10" velocity="3.67"/>
-  </joint>
     <link name="end">
     </link>
@@ -200,7 +176,36 @@
     <joint name="end" type="fixed">
       <origin xyz="${wrist_length} 0 0" rpy="0 ${M_PI/2} 0"/>
-      <parent link="lidar"/>
+      <parent link="gripper_base"/>
       <child link="end"/>
     </joint>
+ <link name="hokuyo">
+    <inertial>
+      <mass value="1e-5"/>
+      <origin xyz="0 0 0" rpy="0 0 0"/>
+      <inertia
+        ixx="1e-8" ixy="0.0" ixz="0.0"
+        iyy="1e-8" iyz="0.0"
+        izz="1e-8"
+      />
+    </inertial>
+    <collision>
+      <origin xyz="0 0 0" rpy="0 0 0"/>
+      <geometry>
+        <box size="0.01 0.01 0.01"/>
+      </geometry>
+    </collision>
+    <visual>
+      <origin xyz="0 0 0" rpy="0 0 0"/>
+      <geometry>
+        <mesh filename="package://al5d_description/meshes/hokuyo.dae"/>
+      </geometry>
+    </visual>
+  </link>
+  <joint name="hokuyo_joint" type="fixed">
+    <origin xyz="0 0 0" rpy="0 0 0" />
+    <parent link="gripper_base"/>
+    <child link="hokuyo" />
+    <axis xyz="0 1 0"/>
+  </joint>
   <gazebo>
     <plugin name="gazebo_ros_control" filename="libgazebo_ros_control.so">

File: al5d_description/urdf/transmissions_lidar.urdf.xacro (robot description, xacro)
@@ -19,12 +19,10 @@
   <xacro:al5d_transmission name="wrist_tilt" />
   <xacro:al5d_transmission name="wrist_rotate" />
-  <xacro:al5d_transmission name="open_gripperright" />
-  <xacro:al5d_transmission name="open_gripperleft" />
-  <!-- hokuyo -->
-<gazebo reference="hokuyo">
+  <xacro:al5d_transmission name="lidar_rotate" />
+<gazebo reference="lidar">
     <sensor type="ray" name="head_hokuyo_sensor">
-      <pose>0 0 0 0 0 0</pose>
+      <pose>0.0 0 0 0 0 0</pose>
       <visualize>true</visualize>
-      <update_rate>40</update_rate>
+      <update_rate>200</update_rate>
       <ray>
         <scan>
@@ -37,5 +35,5 @@
         </scan>
         <range>
-          <min>0.01</min>
+          <min>0.04</min>
           <max>10.0</max>
           <resolution>0.01</resolution>
