Commit message: first commit with meshes from solidworks

File: al5d_description/urdf/al5d_simple.xacro (robot description, xacro)
@@ -27,16 +27,17 @@
     <link name="base">
       <visual>
-        <geometry>
-          <mesh filename="package://al5d_description/mesh/base/Base.STL"/>
-        </geometry>
-        <!-- <material name="silver">
-          <color rgba="0.2 0.2 0.2 0.85"/>
-        </material> -->
-      </visual>
-      <collision>
         <origin xyz="0 0 ${base_height/2}" rpy="0 0 0"/>
         <geometry>
           <cylinder length="${base_height}" radius="${base_radius}"/>
         </geometry>
+        <material name="black">
+          <color rgba="0 0 0 0.85"/>
+        </material>
+      </visual>
+      <collision>
+        <origin xyz="0 0 ${base_height/2}" rpy="0 0 0"/>
+        <geometry>
+          <cylinder length="${base_height}" radius="${base_radius}"/>
+        </geometry>
       </collision>
       <xacro:insert_block name="inertia_block" />
@@ -44,6 +45,24 @@
     <link name="upper_base">
       <visual>
-        <geometry>
-          <mesh filename="package://al5d_description/mesh/upper_base/Waist - HS805BB-1.STL"/>
+	<origin xyz="0 0 ${(upper_base_height - base_height - 0.02)/2 + base_height + 0.02}" rpy="0 0 0"/>
+        <geometry>
+          <cylinder length="${upper_base_height - base_height - 0.02}" radius="${base_radius}"/>
+        </geometry>
+        <material name="black">
+        </material>
+      </visual>
+      <collision>
+	<origin xyz="0 0 ${(upper_base_height - base_height - 0.02)/2 + base_height + 0.02}" rpy="0 0 0"/>
+        <geometry>
+          <cylinder length="${upper_base_height - base_height - 0.02}" radius="${base_radius}"/>
+        </geometry>
+      </collision>
+      <xacro:insert_block name="inertia_block" />
+    </link>
+    <link name="upper_arm">
+      <visual>
+        <origin xyz="${upper_arm_length/2} 0 0" rpy="0 0 0"/>
+        <geometry>
+          <box size="${upper_arm_length} ${upper_arm_width} ${upper_arm_width}"/>
         </geometry>
         <material name="silver">
@@ -51,85 +70,37 @@
         </material>
       </visual>
-      <visual>
-        <geometry>
-          <mesh filename="package://al5d_description/mesh/upper_base/Waist - Turntable-1.STL"/>
+      <collision>
+        <origin xyz="${upper_arm_length/2} 0 0" rpy="0 0 0"/>
+        <geometry>
+          <box size="${upper_arm_length} ${upper_arm_width} ${upper_arm_width}"/>
+        </geometry>
+      </collision>
+      <xacro:insert_block name="inertia_block" />
+    </link>
+    <link name="lower_arm">
+      <visual>
+        <origin xyz="${lower_arm_length/2} 0 0" rpy="0 0 0"/>
+        <geometry>
+          <box size="${lower_arm_length} ${lower_arm_width} ${lower_arm_width}"/>
+        </geometry>
+        <material name="blue">
+          <color rgba="0.4 0.4 1 0.85"/>
+        </material>
+      </visual>
+      <collision>
+        <origin xyz="${lower_arm_length/2} 0 0" rpy="0 0 0"/>
+        <geometry>
+          <box size="${lower_arm_length} ${lower_arm_width} ${lower_arm_width}"/>
+        </geometry>
+      </collision>
+      <xacro:insert_block name="inertia_block" />
+    </link>
+    <link name="wrist">
+      <visual>
+        <origin xyz="${wrist_length/2} 0 0" rpy="0 0 0"/>
+        <geometry>
+          <box size="${wrist_length} ${wrist_width} ${wrist_width}"/>
         </geometry>
         <material name="silver">
-          <color rgba="0.8 0.8 0.8 0.85"/>
-        </material>
-      </visual>
-      <collision>
-	<origin xyz="0 0 ${(upper_base_height - base_height - 0.02)/2 + base_height + 0.02}" rpy="0 0 0"/>
-        <geometry>
-          <cylinder length="${upper_base_height - base_height - 0.02}" radius="${base_radius}"/>
-        </geometry>
-      </collision>
-      <xacro:insert_block name="inertia_block" />
-    </link>
-    <link name="upper_arm">
-      <visual>
-        <geometry>
-          <mesh filename="package://al5d_description/mesh/upper_arm/UpperArm - Bracket-1.STL"/>
-        </geometry>
-        <material name="silver">
-          <color rgba="0.8 0.8 0.8 0.85"/>
-        </material>
-      </visual>
-      <visual>
-        <geometry>
-          <mesh filename="package://al5d_description/mesh/upper_arm/UpperArm - Bracket-2.STL"/>
-        </geometry>
-        <material name="silver">
-          <color rgba="0.8 0.8 0.8 0.85"/>
-        </material>
-      </visual>
-      <collision>
-        <origin xyz="${upper_arm_length/2} 0 0" rpy="0 0 0"/>
-        <geometry>
-          <box size="${upper_arm_length} ${upper_arm_width} ${upper_arm_width}"/>
-        </geometry>
-      </collision>
-      <xacro:insert_block name="inertia_block" />
-    </link>
-    <link name="lower_arm">
-      <visual>
-        <geometry>
-          <mesh filename="package://al5d_description/mesh/lower_arm/LowerArm - HS422-1.STL"/>
-        </geometry>
-        <material name="silver">
-          <color rgba="0.8 0.8 0.8 0.85"/>
-        </material>
-      </visual>
-      <visual>
-        <geometry>
-          <mesh filename="package://al5d_description/mesh/lower_arm/LowerArm - HS805BB-1.STL"/>
-        </geometry>
-        <material name="silver">
-          <color rgba="0.8 0.8 0.8 0.85"/>
-        </material>
-      </visual>
-      <visual>
-        <geometry>
-          <mesh filename="package://al5d_description/mesh/lower_arm/LowerArm - Rod-1.STL"/>
-        </geometry>
-        <material name="silver">
-          <color rgba="0.8 0.8 0.8 0.85"/>
-        </material>
-      </visual>
-      <collision>
-        <origin xyz="${lower_arm_length/2} 0 0" rpy="0 0 0"/>
-        <geometry>
-          <box size="${lower_arm_length} ${lower_arm_width} ${lower_arm_width}"/>
-        </geometry>
-      </collision>
-      <xacro:insert_block name="inertia_block" />
-    </link>
-    <link name="wrist">
-      <visual>
-        <geometry>
-          <mesh filename="package://al5d_description/mesh/wrist/WristLink.STL"/>
-        </geometry>
-        <material name="silver">
-          <color rgba="0.8 0.8 0.8 0.85"/>
         </material>
       </visual>
@@ -144,17 +115,10 @@
     <link name="gripper_base">
       <visual>
-        <geometry>
-          <mesh filename="package://al5d_description/mesh/gripper_base/Gripper - WristTurn-1.STL"/>
-        </geometry>
-        <material name="silver">
-          <color rgba="0.8 0.8 0.8 0.85"/>
-        </material>
-      </visual>
-      <visual>
-        <geometry>
-          <mesh filename="package://al5d_description/mesh/gripper_base/Gripper - GripperBase-1.STL"/>
-        </geometry>
-        <material name="silver">
-          <color rgba="0.8 0.8 0.8 0.85"/>
+	<origin xyz="${gripper_height/2} 0 0" rpy="0 0 0"/>
+        <geometry>
+          <box size="${gripper_height} ${gripper_height} ${gripper_width}"/>
+        </geometry>
+        <material name="red">
+          <color rgba="1 0.3 0.3 0.85"/>
         </material>
       </visual>
@@ -169,9 +133,10 @@
     <link name="gripper_rightfinger">
       <visual>
-        <geometry>
-          <mesh filename="package://al5d_description/mesh/right_finger/RightFinger.STL"/>
-        </geometry>
-        <material name="silver">
-          <color rgba="0.8 0.8 0.8 0.85"/>
+	<origin xyz="${finger_length/2} 0 0" rpy="0 0 0"/>
+        <geometry>
+          <box size="${finger_length} ${gripper_height} ${gripper_height}"/>
+        </geometry>
+        <material name="red">
+          <color rgba="1 0.3 0.3 0.85"/>
         </material>
       </visual>
@@ -189,7 +154,11 @@
     <link name="gripper_leftfinger">
       <visual>
-        <geometry>
-          <mesh filename="package://al5d_description/mesh/left_finger/LeftFinger.STL"/>
-        </geometry>
+	<origin xyz="${finger_length/2} 0 0" rpy="0 0 0"/>
+        <geometry>
+          <box size="${finger_length} ${gripper_height} ${gripper_height}"/>
+        </geometry>
+        <material name="red">
+          <color rgba="1 0.3 0.3 0.85"/>
+        </material>
       </visual>
       <collision>
@@ -279,45 +248,33 @@
     </plugin>
   </gazebo>
+  <gazebo reference="end">
+    <material value="Gazebo/Red" />
+  </gazebo>
+  <gazebo reference="base_rotate">
+    <material value="Gazebo/Grey" />
+  </gazebo>
   <gazebo reference="shoulder_tilt">
+    <material value="Gazebo/Grey" />
     <turnGravityOff>true</turnGravityOff>
   </gazebo>
   <gazebo reference="elbow_tilt">
+    <material value="Gazebo/Grey" />
     <turnGravityOff>true</turnGravityOff>
   </gazebo>
   <gazebo reference="wrist_tilt">
+    <material value="Gazebo/Grey" />
     <turnGravityOff>true</turnGravityOff>
   </gazebo>
   <gazebo reference="wrist_rotate">
+    <material value="Gazebo/Grey" />
     <turnGravityOff>true</turnGravityOff>
   </gazebo>
   <gazebo reference="open_gripperright">
+    <material value="Gazebo/Grey" />
     <turnGravityOff>true</turnGravityOff>
   </gazebo>
   <gazebo reference="open_gripperleft">
-    <turnGravityOff>true</turnGravityOff>
-  </gazebo>
-  <gazebo reference="base">
-    <material>Gazebo/DarkGrey</material>
-  </gazebo>
-  <!-- <gazebo reference="upper_base">
-    <material>Gazebo/DarkGrey</material>
-  </gazebo> -->
-  <gazebo reference="upper_arm">
-    <material>Gazebo/DarkGrey</material>
-  </gazebo>
-  <!-- <gazebo reference="lower_arm">
-    <material>Gazebo/DarkGrey</material>
-  </gazebo> -->
-  <gazebo reference="wrist">
-    <material>Gazebo/DarkGrey</material>
-  </gazebo>
-  <!-- <gazebo reference="gripper_base">
-    <material>Gazebo/DarkGrey</material>
-  </gazebo> -->
-  <gazebo reference="gripper_leftfinger">
-    <material>Gazebo/DarkGrey</material>
-  </gazebo>
-  <gazebo reference="gripper_rightfinger">
-    <material>Gazebo/DarkGrey</material>
+    <material value="Gazebo/Grey" />
+    <turnGravityOff>true</turnGravityOff>
   </gazebo>
 </robot>
