Commit message: Working launch file with platforms, turntable, and objects (not random)

File: al5d_description/urdf/turntable.xacro (robot description, xacro)
@@ -71,5 +71,5 @@
   </gazebo>
   <gazebo reference="upper_base">
-    <material>Gazebo/Wood</material>
+    <material>Gazebo/DarkGrey</material>
   </gazebo>
 </robot>

Commit message: functional code for final project with object and opponent sensing

File: al5d_description/urdf/turntable.xacro (robot description, xacro)
@@ -15,13 +15,13 @@
     <link name="base">
       <visual>
-        <origin xyz="0 0 ${.0532/2}" rpy="0 0 0"/>
+        <origin xyz="0 0 ${.04/2}" rpy="0 0 0"/>
         <geometry>
-          <cylinder length=".0532" radius="${base_radius}"/>
+          <cylinder length=".04" radius="${base_radius}"/>
         </geometry>
       </visual>
       <collision>
-        <origin xyz="0 0 ${.0532/2}" rpy="0 0 0"/>
+        <origin xyz="0 0 ${.04/2}" rpy="0 0 0"/>
         <geometry>
-          <cylinder length=".0532" radius="${base_radius}"/>
+          <cylinder length=".04" radius="${base_radius}"/>
         </geometry>
       </collision>
@@ -33,13 +33,13 @@
     <link name="upper_base">
       <visual>
-	      <origin xyz="0 0 .0582" rpy="0 0 0"/>
+	      <origin xyz="0 0 .045" rpy="0 0 0"/>
         <geometry>
-          <cylinder length=".004" radius="${base_radius}"/>
+          <cylinder length=".01" radius="${base_radius}"/>
         </geometry>
       </visual>
       <collision>
-	      <origin xyz="0 0 .0582" rpy="0 0 0"/>
+	      <origin xyz="0 0 .045" rpy="0 0 0"/>
         <geometry>
-          <cylinder length=".004" radius="${base_radius}"/>
+          <cylinder length=".01" radius="${base_radius}"/>
         </geometry>
       </collision>
