Commit message: fixing cad to match dimensions in sim

File: al5d_description/urdf/al5d_cad.xacro (robot description, xacro)
@@ -15,7 +15,10 @@
     <xacro:property name="wrist_width" value="0.025" />
     <xacro:property name="gripper_width" value="0.05" />
-    <xacro:property name="gripper_height" value="0.01" />
+    <xacro:property name="gripper_height" value="0.021" />
+    <!-- <xacro:property name="gripper_height" value="0.01" /> -->
     <xacro:property name="finger_length" value="0.04" />
     <xacro:property name="point" value="0.003" />
+    <xacro:property name="axis_length" value="0.03" />
+    <xacro:property name="axis_width" value="0.001" />
     <xacro:property name="inertia_block">
       <inertial>
@@ -60,5 +63,5 @@
       </visual>
       <collision>
-	<origin xyz="0 0 ${(upper_base_height - base_height - 0.02)/2 + base_height + 0.02}" rpy="0 0 0"/>
+	       <origin xyz="0 0 ${(upper_base_height - base_height - 0.02)/2 + base_height + 0.02}" rpy="0 0 0"/>
         <geometry>
           <cylinder length="${upper_base_height - base_height - 0.02}" radius="${base_radius}"/>
@@ -117,9 +120,15 @@
         </material>
       </visual>
-      <collision>
+      <!-- <visual>
         <origin xyz="${lower_arm_length/2} 0 0" rpy="0 0 0"/>
         <geometry>
           <box size="${lower_arm_length} ${lower_arm_width} ${lower_arm_width}"/>
         </geometry>
+      </visual> -->
+      <collision>
+        <origin xyz="${lower_arm_length/2} 0 0" rpy="0 0 0"/>
+        <geometry>
+          <box size="${lower_arm_length} ${lower_arm_width} ${lower_arm_width}"/>
+        </geometry>
       </collision>
       <xacro:insert_block name="inertia_block" />
@@ -134,9 +143,15 @@
         </material>
       </visual>
-      <collision>
+      <!-- <visual>
         <origin xyz="${wrist_length/2} 0 0" rpy="0 0 0"/>
         <geometry>
           <box size="${wrist_length} ${wrist_width} ${wrist_width}"/>
         </geometry>
+      </visual> -->
+      <collision>
+        <origin xyz="${wrist_length/2} 0 0" rpy="0 0 0"/>
+        <geometry>
+          <box size="${wrist_length} ${wrist_width} ${wrist_width}"/>
+        </geometry>
       </collision>
       <xacro:insert_block name="inertia_block" />
@@ -147,7 +162,4 @@
           <mesh filename="package://al5d_description/mesh/gripper_base/Gripper - WristTurn-1.STL"/>
         </geometry>
-        <material name="silver">
-          <color rgba="0.8 0.8 0.8 0.85"/>
-        </material>
       </visual>
       <visual>
@@ -155,13 +167,16 @@
           <mesh filename="package://al5d_description/mesh/gripper_base/Gripper - GripperBase-1.STL"/>
         </geometry>
-        <material name="silver">
-          <color rgba="0.8 0.8 0.8 0.85"/>
-        </material>
-      </visual>
-      <collision>
-        <origin xyz="${gripper_width/2} 0 0" rpy="0 0 0"/>
+      </visual>
+      <!-- <visual>
+	      <origin xyz="${gripper_height/2} 0 0" rpy="0 0 0"/>
         <geometry>
           <box size="${gripper_height} ${gripper_height} ${gripper_width}"/>
         </geometry>
+      </visual> -->
+      <collision>
+        <origin xyz="${gripper_width/2} 0 0" rpy="0 0 0"/>
+        <geometry>
+          <box size="${gripper_height} ${gripper_height} ${gripper_width}"/>
+        </geometry>
       </collision>
       <xacro:insert_block name="inertia_block" />
@@ -172,12 +187,15 @@
           <mesh filename="package://al5d_description/mesh/right_finger/RightFinger.STL"/>
         </geometry>
-        <material name="silver">
-          <color rgba="0.8 0.8 0.8 0.85"/>
-        </material>
-      </visual>
-      <collision>
-        <origin xyz="${gripper_width/2} 0 0" rpy="0 0 0"/>
-        <geometry>
-		<box size="${gripper_width} ${gripper_height} ${gripper_height}"/>
+      </visual>
+      <!-- <visual>
+        <origin xyz="${gripper_width/2} 0 0" rpy="0 0 0"/>
+        <geometry>
+		      <box size="${gripper_width} ${gripper_height} ${gripper_height}"/>
+        </geometry>
+      </visual> -->
+      <collision>
+        <origin xyz="${gripper_width/2} 0 0" rpy="0 0 0"/>
+        <geometry>
+		      <box size="${gripper_width} ${gripper_height} ${gripper_height}"/>
         </geometry>
       </collision>
@@ -193,4 +211,10 @@
         </geometry>
       </visual>
+      <!-- <visual>
+        <origin xyz="${gripper_width/2} 0 0" rpy="0 0 0"/>
+        <geometry>
+          <box size="${gripper_width} ${gripper_height} ${gripper_height}"/>
+        </geometry>
+      </visual> -->
       <collision>
         <origin xyz="${gripper_width/2} 0 0" rpy="0 0 0"/>
@@ -207,10 +231,31 @@
       <!-- <visual>
         <geometry>
-          <box size="${point} ${point} ${point}"/>
-        </geometry>
-        <material name="red">
-          <color rgba="1 0.3 0.3 0.85"/>
-        </material>
-      </visual> -->
+          <sphere radius=".001" />
+        </geometry>
+      </visual> -->
+    </link>
+    <link name="xaxis">
+      <visual>
+        <origin xyz="${axis_length/2} 0 0" rpy="0 0 0"/>
+        <geometry>
+          <box size="${axis_length} ${axis_width} ${axis_width}"/>
+        </geometry>
+      </visual>
+    </link>
+    <link name="yaxis">
+      <visual>
+        <origin xyz="0 ${axis_length/2} 0" rpy="0 0 0"/>
+        <geometry>
+          <box size="${axis_width} ${axis_length} ${axis_width}"/>
+        </geometry>
+      </visual>
+    </link>
+    <link name="zaxis">
+      <visual>
+        <origin xyz="0 0 ${axis_length/2}" rpy="0 0 0"/>
+        <geometry>
+          <box size="${axis_width} ${axis_width} ${axis_length}"/>
+        </geometry>
+      </visual>
     </link>
     <!-- joints -->
@@ -274,4 +319,19 @@
       <child link="end"/>
     </joint>
+    <joint name="axis1" type="fixed">
+      <origin xyz="0 0 0" rpy="0 0 0"/>
+      <parent link="end"/>
+      <child link="xaxis"/>
+    </joint>
+    <joint name="axis2" type="fixed">
+      <origin xyz="0 0 0" rpy="0 0 0"/>
+      <parent link="end"/>
+      <child link="yaxis"/>
+    </joint>
+    <joint name="axis3" type="fixed">
+      <origin xyz="0 0 0" rpy="0 0 0"/>
+      <parent link="end"/>
+      <child link="zaxis"/>
+    </joint>
   <gazebo>
     <plugin name="gazebo_ros_control" filename="libgazebo_ros_control.so">
@@ -279,45 +339,42 @@
     </plugin>
   </gazebo>
-  <gazebo reference="shoulder_tilt">
-    <turnGravityOff>true</turnGravityOff>
-  </gazebo>
-  <gazebo reference="elbow_tilt">
-    <turnGravityOff>true</turnGravityOff>
-  </gazebo>
-  <gazebo reference="wrist_tilt">
-    <turnGravityOff>true</turnGravityOff>
-  </gazebo>
-  <gazebo reference="wrist_rotate">
-    <turnGravityOff>true</turnGravityOff>
-  </gazebo>
-  <gazebo reference="open_gripperright">
-    <turnGravityOff>true</turnGravityOff>
-  </gazebo>
-  <gazebo reference="open_gripperleft">
-    <turnGravityOff>true</turnGravityOff>
-  </gazebo>
   <gazebo reference="base">
     <material>Gazebo/DarkGrey</material>
-  </gazebo>
-  <!-- <gazebo reference="upper_base">
-    <material>Gazebo/DarkGrey</material>
-  </gazebo> -->
+    <turnGravityOff>true</turnGravityOff>
+  </gazebo>
+  <gazebo reference="upper_base">
+    <turnGravityOff>true</turnGravityOff>
+  </gazebo>
   <gazebo reference="upper_arm">
-    <material>Gazebo/DarkGrey</material>
-  </gazebo>
-  <!-- <gazebo reference="lower_arm">
-    <material>Gazebo/DarkGrey</material>
-  </gazebo> -->
+    <turnGravityOff>true</turnGravityOff>
+    <material>Gazebo/DarkGrey</material>
+  </gazebo>
+  <gazebo reference="lower_arm">
+    <turnGravityOff>true</turnGravityOff>
+  </gazebo>
   <gazebo reference="wrist">
-    <material>Gazebo/DarkGrey</material>
-  </gazebo>
-  <!-- <gazebo reference="gripper_base">
-    <material>Gazebo/DarkGrey</material>
-  </gazebo> -->
+    <turnGravityOff>true</turnGravityOff>
+    <material>Gazebo/DarkGrey</material>
+  </gazebo>
+  <gazebo reference="gripper_base">
+    <turnGravityOff>true</turnGravityOff>
+  </gazebo>
   <gazebo reference="gripper_leftfinger">
+    <turnGravityOff>true</turnGravityOff>
     <material>Gazebo/DarkGrey</material>
   </gazebo>
   <gazebo reference="gripper_rightfinger">
-    <material>Gazebo/DarkGrey</material>
+    <turnGravityOff>true</turnGravityOff>
+    <material>Gazebo/DarkGrey</material>
+  </gazebo>
+  <gazebo reference="end"></gazebo>
+  <gazebo reference="xaxis">
+    <material>Gazebo/RedTransparentOverlay</material>
+  </gazebo>
+  <gazebo reference="yaxis">
+    <material>Gazebo/GreenTransparentOverlay</material>
+  </gazebo>
+  <gazebo reference="zaxis">
+    <material>Gazebo/BlueTransparentOverlay</material>
   </gazebo>
 </robot>

File: al5d_description/urdf/al5d_simple.xacro (robot description, xacro)
@@ -115,5 +115,5 @@
     <link name="gripper_base">
       <visual>
-	<origin xyz="${gripper_height/2} 0 0" rpy="0 0 0"/>
+	      <origin xyz="${gripper_height/2} 0 0" rpy="0 0 0"/>
         <geometry>
           <box size="${gripper_height} ${gripper_height} ${gripper_width}"/>

Commit message: New visualization ready to give to students

File: al5d_description/urdf/al5d_cad.xacro (robot description, xacro)
@@ -301,5 +301,6 @@
     </joint>
     <joint name="open_gripperright" type="prismatic">
-      <origin xyz="${gripper_height} 0 0.03" rpy="0 0 0"/>
+      <origin xyz="${gripper_height} 0 0.023" rpy="0 0 0"/>
+      <origin xyz="${gripper_height} 0 0" rpy="0 0 0"/>
       <parent link="gripper_base"/>
       <child link="gripper_rightfinger"/>
@@ -308,5 +309,5 @@
     </joint>
     <joint name="open_gripperleft" type="prismatic">
-      <origin xyz="${gripper_height} 0 -0.03" rpy="0 0 0"/>
+      <origin xyz="${gripper_height} 0 -0.023" rpy="0 0 0"/>
       <parent link="gripper_base"/>
       <child link="gripper_leftfinger"/>
@@ -368,13 +369,18 @@
     <material>Gazebo/DarkGrey</material>
   </gazebo>
-  <gazebo reference="end"></gazebo>
+  <gazebo reference="end">
+    <turnGravityOff>true</turnGravityOff>
+  </gazebo>
   <gazebo reference="xaxis">
     <material>Gazebo/RedTransparentOverlay</material>
+    <turnGravityOff>true</turnGravityOff>
   </gazebo>
   <gazebo reference="yaxis">
     <material>Gazebo/GreenTransparentOverlay</material>
+    <turnGravityOff>true</turnGravityOff>
   </gazebo>
   <gazebo reference="zaxis">
     <material>Gazebo/BlueTransparentOverlay</material>
+    <turnGravityOff>true</turnGravityOff>
   </gazebo>
 </robot>

Commit message: Major updates to arm controller including
- ROS messaging API to gut MATLAB class
- Velocity control
- is_stopped flag

File: al5d_description/urdf/al5d_cad.xacro (robot description, xacro)
@@ -30,7 +30,11 @@
     <link name="base">
       <visual>
-        <geometry>
+        <origin xyz="0 0 ${base_height/2}" rpy="0 0 0"/>
+        <geometry>
+          <cylinder length="${base_height}" radius="${base_radius}"/>
+        </geometry>
+        <!-- <geometry>
           <mesh filename="package://al5d_description/mesh/base/Base.STL"/>
-        </geometry>
+        </geometry> -->
         <!-- <material name="silver">
           <color rgba="0.2 0.2 0.2 0.85"/>
@@ -184,6 +188,7 @@
     <link name="gripper_rightfinger">
       <visual>
-        <geometry>
-          <mesh filename="package://al5d_description/mesh/right_finger/RightFinger.STL"/>
+        <origin xyz="${gripper_width/4} 0 0" rpy="0 0 0"/>
+        <geometry>
+          <box size="${gripper_width/2} ${gripper_height} ${gripper_height/4}"/>
         </geometry>
       </visual>
@@ -195,7 +200,7 @@
       </visual> -->
       <collision>
-        <origin xyz="${gripper_width/2} 0 0" rpy="0 0 0"/>
-        <geometry>
-		      <box size="${gripper_width} ${gripper_height} ${gripper_height}"/>
+        <origin xyz="${gripper_width/4} 0 0" rpy="0 0 0"/>
+        <geometry>
+          <box size="${gripper_width/2} ${gripper_height} ${gripper_height/4}"/>
         </geometry>
       </collision>
@@ -206,20 +211,24 @@
     </link>
     <link name="gripper_leftfinger">
-      <visual>
+      <!-- <visual>
         <geometry>
           <mesh filename="package://al5d_description/mesh/left_finger/LeftFinger.STL"/>
         </geometry>
-      </visual>
-      <!-- <visual>
-        <origin xyz="${gripper_width/2} 0 0" rpy="0 0 0"/>
+      </visual> -->
+      <visual>
+        <origin xyz="${gripper_width/4} 0 0" rpy="0 0 0"/>
+        <geometry>
+          <box size="${gripper_width/2} ${gripper_height} ${gripper_height/4}"/>
+        </geometry>
+      </visual>
+      <collision>
+        <origin xyz="${gripper_width/4} 0 0" rpy="0 0 0"/>
+        <geometry>
+          <box size="${gripper_width/2} ${gripper_height} ${gripper_height/4}"/>
+        </geometry>
+        <!-- <origin xyz="${gripper_width/2} 0 0" rpy="0 0 0"/>
         <geometry>
           <box size="${gripper_width} ${gripper_height} ${gripper_height}"/>
-        </geometry>
-      </visual> -->
-      <collision>
-        <origin xyz="${gripper_width/2} 0 0" rpy="0 0 0"/>
-        <geometry>
-          <box size="${gripper_width} ${gripper_height} ${gripper_height}"/>
-        </geometry>
+        </geometry> -->
       </collision>
       <inertial>
@@ -343,4 +352,5 @@
     <material>Gazebo/DarkGrey</material>
     <turnGravityOff>true</turnGravityOff>
+    <!-- <self_collide>1</self_collide> -->
   </gazebo>
   <gazebo reference="upper_base">
@@ -364,8 +374,10 @@
     <turnGravityOff>true</turnGravityOff>
     <material>Gazebo/DarkGrey</material>
+    <!-- <self_collide>1</self_collide> -->
   </gazebo>
   <gazebo reference="gripper_rightfinger">
     <turnGravityOff>true</turnGravityOff>
     <material>Gazebo/DarkGrey</material>
+    <!-- <self_collide>1</self_collide> -->
   </gazebo>
   <gazebo reference="end">

Commit message: fixing broken base visualization

File: al5d_description/urdf/al5d_cad.xacro (robot description, xacro)
@@ -30,14 +30,11 @@
     <link name="base">
       <visual>
-        <origin xyz="0 0 ${base_height/2}" rpy="0 0 0"/>
+        <!-- <origin xyz="0 0 ${base_height/2}" rpy="0 0 0"/>
         <geometry>
           <cylinder length="${base_height}" radius="${base_radius}"/>
-        </geometry>
-        <!-- <geometry>
+        </geometry> -->
+        <geometry>
           <mesh filename="package://al5d_description/mesh/base/Base.STL"/>
-        </geometry> -->
-        <!-- <material name="silver">
-          <color rgba="0.2 0.2 0.2 0.85"/>
-        </material> -->
+        </geometry>
       </visual>
       <collision>
