Commit message: updated collision geometry, visuals using basic commands, and colors

File: al5d_description/urdf/al5d_cad.xacro (robot description, xacro)
@@ -16,5 +16,4 @@
     <xacro:property name="gripper_width" value="0.05" />
     <xacro:property name="gripper_height" value="0.021" />
-    <!-- <xacro:property name="gripper_height" value="0.01" /> -->
     <xacro:property name="finger_length" value="0.04" />
     <xacro:property name="point" value="0.003" />
@@ -30,16 +29,13 @@
     <link name="base">
       <visual>
-        <!-- <origin xyz="0 0 ${base_height/2}" rpy="0 0 0"/>
-        <geometry>
-          <cylinder length="${base_height}" radius="${base_radius}"/>
-        </geometry> -->
-        <geometry>
-          <mesh filename="package://al5d_description/mesh/base/Base.STL"/>
-        </geometry>
-      </visual>
-      <collision>
-        <origin xyz="0 0 ${base_height/2}" rpy="0 0 0"/>
-        <geometry>
-          <cylinder length="${base_height}" radius="${base_radius}"/>
+        <origin xyz="0 0 ${.0532/2}" rpy="0 0 0"/>
+        <geometry>
+          <cylinder length=".0532" radius="${base_radius}"/>
+        </geometry>
+      </visual>
+      <collision>
+        <origin xyz="0 0 ${.0532/2}" rpy="0 0 0"/>
+        <geometry>
+          <cylinder length=".0532" radius="${base_radius}"/>
         </geometry>
       </collision>
@@ -48,23 +44,25 @@
     <link name="upper_base">
       <visual>
-        <geometry>
-          <mesh filename="package://al5d_description/mesh/upper_base/Waist - HS805BB-1.STL"/>
-        </geometry>
-        <material name="silver">
-          <color rgba="0.8 0.8 0.8 0.85"/>
-        </material>
-      </visual>
-      <visual>
-        <geometry>
-          <mesh filename="package://al5d_description/mesh/upper_base/Waist - Turntable-1.STL"/>
-        </geometry>
-        <material name="silver">
-          <color rgba="0.8 0.8 0.8 0.85"/>
-        </material>
-      </visual>
-      <collision>
-	       <origin xyz="0 0 ${(upper_base_height - base_height - 0.02)/2 + base_height + 0.02}" rpy="0 0 0"/>
-        <geometry>
-          <cylinder length="${upper_base_height - base_height - 0.02}" radius="${base_radius}"/>
+	      <origin xyz="0 0 .0582" rpy="0 0 0"/>
+        <geometry>
+          <cylinder length=".004" radius="${base_radius}"/>
+        </geometry>
+      </visual>
+      <visual>
+	      <origin xyz="-.01487 0 .0752" rpy="0 0 0"/>
+        <geometry>
+          <box size=".06985 .0508 .030"/>
+        </geometry>
+      </visual>
+      <collision>
+	      <origin xyz="0 0 .0582" rpy="0 0 0"/>
+        <geometry>
+          <cylinder length=".004" radius="${base_radius}"/>
+        </geometry>
+      </collision>
+      <collision>
+	      <origin xyz="-.01487 0 .0752" rpy="0 0 0"/>
+        <geometry>
+          <box size=".06985 .0508 .030"/>
         </geometry>
       </collision>
@@ -76,7 +74,4 @@
           <mesh filename="package://al5d_description/mesh/upper_arm/UpperArm - Bracket-1.STL"/>
         </geometry>
-        <material name="silver">
-          <color rgba="0.8 0.8 0.8 0.85"/>
-        </material>
       </visual>
       <visual>
@@ -84,12 +79,21 @@
           <mesh filename="package://al5d_description/mesh/upper_arm/UpperArm - Bracket-2.STL"/>
         </geometry>
-        <material name="silver">
-          <color rgba="0.8 0.8 0.8 0.85"/>
-        </material>
       </visual>
       <collision>
         <origin xyz="${upper_arm_length/2} 0 0" rpy="0 0 0"/>
         <geometry>
-          <box size="${upper_arm_length} ${upper_arm_width} ${upper_arm_width}"/>
+          <box size=".02 .020 .068"/>
+        </geometry>
+      </collision>
+      <collision>
+        <origin xyz="${upper_arm_length/2} 0 .033" rpy="0 0 0"/>
+        <geometry>
+          <box size=".166 .020 .002"/>
+        </geometry>
+      </collision>
+      <collision>
+        <origin xyz="${upper_arm_length/2} 0 -.033" rpy="0 0 0"/>
+        <geometry>
+          <box size=".166 .020 .002"/>
         </geometry>
       </collision>
@@ -98,37 +102,37 @@
     <link name="lower_arm">
       <visual>
-        <geometry>
-          <mesh filename="package://al5d_description/mesh/lower_arm/LowerArm - HS422-1.STL"/>
-        </geometry>
-        <material name="silver">
-          <color rgba="0.8 0.8 0.8 0.85"/>
-        </material>
-      </visual>
-      <visual>
-        <geometry>
-          <mesh filename="package://al5d_description/mesh/lower_arm/LowerArm - HS805BB-1.STL"/>
-        </geometry>
-        <material name="silver">
-          <color rgba="0.8 0.8 0.8 0.85"/>
-        </material>
-      </visual>
-      <visual>
-        <geometry>
-          <mesh filename="package://al5d_description/mesh/lower_arm/LowerArm - Rod-1.STL"/>
-        </geometry>
-        <material name="silver">
-          <color rgba="0.8 0.8 0.8 0.85"/>
-        </material>
-      </visual>
-      <!-- <visual>
-        <origin xyz="${lower_arm_length/2} 0 0" rpy="0 0 0"/>
-        <geometry>
-          <box size="${lower_arm_length} ${lower_arm_width} ${lower_arm_width}"/>
-        </geometry>
-      </visual> -->
-      <collision>
-        <origin xyz="${lower_arm_length/2} 0 0" rpy="0 0 0"/>
-        <geometry>
-          <box size="${lower_arm_length} ${lower_arm_width} ${lower_arm_width}"/>
+        <origin xyz="${lower_arm_length/2} 0 0" rpy="0 ${3.14158/2} 0"/>
+        <geometry>
+          <cylinder length="${lower_arm_length}" radius=".00635"/>
+        </geometry>
+      </visual>
+      <visual>
+        <origin xyz="-.01982 0 0" rpy="0 0 0"/>
+        <geometry>
+          <box size=".06985 .030 .0508"/>
+        </geometry>
+      </visual>
+      <visual>
+        <origin xyz=".1759 0 0" rpy="0 0 0"/>
+        <geometry>
+          <box size=".0508 .0279 .0381"/>
+        </geometry>
+      </visual>
+      <collision>
+        <origin xyz="${lower_arm_length/2} 0 0" rpy="0 ${3.14158/2} 0"/>
+        <geometry>
+          <cylinder length="${lower_arm_length}" radius=".00635"/>
+        </geometry>
+      </collision>
+      <collision>
+        <origin xyz="-.01982 0 0" rpy="0 0 0"/>
+        <geometry>
+          <box size=".06985 .030 .0508"/>
+        </geometry>
+      </collision>
+      <collision>
+        <origin xyz=".1759 0 0" rpy="0 0 0"/>
+        <geometry>
+          <box size=".0508 .0279 .0381"/>
         </geometry>
       </collision>
@@ -137,21 +141,37 @@
     <link name="wrist">
       <visual>
-        <geometry>
-          <mesh filename="package://al5d_description/mesh/wrist/WristLink.STL"/>
-        </geometry>
-        <material name="silver">
-          <color rgba="0.8 0.8 0.8 0.85"/>
-        </material>
-      </visual>
-      <!-- <visual>
-        <origin xyz="${wrist_length/2} 0 0" rpy="0 0 0"/>
-        <geometry>
-          <box size="${wrist_length} ${wrist_width} ${wrist_width}"/>
-        </geometry>
-      </visual> -->
-      <collision>
-        <origin xyz="${wrist_length/2} 0 0" rpy="0 0 0"/>
-        <geometry>
-          <box size="${wrist_length} ${wrist_width} ${wrist_width}"/>
+        <origin xyz=".026 0 0" rpy="0 0 0"/>
+        <geometry>
+          <box size=".002 .020 .05788"/>
+        </geometry>
+      </visual>
+      <visual>
+        <origin xyz="${.025-.0377/2} 0 ${.05788/2-.001}" rpy="0 0 0"/>
+        <geometry>
+          <box size="${.0377} .020 .002"/>
+        </geometry>
+      </visual>
+      <visual>
+        <origin xyz="${.025-.0377/2} 0 ${-.05788/2+.001}" rpy="0 0 0"/>
+        <geometry>
+          <box size="${.0377} .020 .002"/>
+        </geometry>
+      </visual>
+      <collision>
+        <origin xyz=".026 0 0" rpy="0 0 0"/>
+        <geometry>
+          <box size=".002 .020 .05788"/>
+        </geometry>
+      </collision>
+      <collision>
+        <origin xyz="${.025-.0377/2} 0 ${.05788/2-.001}" rpy="0 0 0"/>
+        <geometry>
+          <box size="${.0377} .020 .002"/>
+        </geometry>
+      </collision>
+      <collision>
+        <origin xyz="${.025-.0377/2} 0 ${-.05788/2+.001}" rpy="0 0 0"/>
+        <geometry>
+          <box size="${.0377} .020 .002"/>
         </geometry>
       </collision>
@@ -160,23 +180,26 @@
     <link name="gripper_base">
       <visual>
-        <geometry>
-          <mesh filename="package://al5d_description/mesh/gripper_base/Gripper - WristTurn-1.STL"/>
-        </geometry>
-      </visual>
-      <visual>
-        <geometry>
-          <mesh filename="package://al5d_description/mesh/gripper_base/Gripper - GripperBase-1.STL"/>
-        </geometry>
-      </visual>
-      <!-- <visual>
-	      <origin xyz="${gripper_height/2} 0 0" rpy="0 0 0"/>
-        <geometry>
-          <box size="${gripper_height} ${gripper_height} ${gripper_width}"/>
-        </geometry>
-      </visual> -->
-      <collision>
-        <origin xyz="${gripper_width/2} 0 0" rpy="0 0 0"/>
-        <geometry>
-          <box size="${gripper_height} ${gripper_height} ${gripper_width}"/>
+        <origin xyz=".014 0 0" rpy="0 0 0"/>
+        <geometry>
+          <box size=".014 .018 .05"/>
+        </geometry>
+      </visual>
+      <visual>
+        <origin xyz="0 0 0" rpy="0 ${3.14159/2} 0"/>
+        <geometry>
+          <cylinder length=".014" radius=".009"/>
+        </geometry>
+      </visual>
+      <collision>
+        <origin xyz=".014 0 0" rpy="0 0 0"/>
+        <geometry>
+          <box size=".014 .018 .05"/>
+        </geometry>
+      </collision>
+      <collision>
+        <origin xyz="0 0 0" rpy="0 ${3.14159/2} 0"/>
+        <geometry>
+          <!-- shorter to avoid numerical issues -->
+          <cylinder length=".013" radius=".009"/>
         </geometry>
       </collision>
@@ -208,9 +231,4 @@
     </link>
     <link name="gripper_leftfinger">
-      <!-- <visual>
-        <geometry>
-          <mesh filename="package://al5d_description/mesh/left_finger/LeftFinger.STL"/>
-        </geometry>
-      </visual> -->
       <visual>
         <origin xyz="${gripper_width/4} 0 0" rpy="0 0 0"/>
@@ -224,8 +242,4 @@
           <box size="${gripper_width/2} ${gripper_height} ${gripper_height/4}"/>
         </geometry>
-        <!-- <origin xyz="${gripper_width/2} 0 0" rpy="0 0 0"/>
-        <geometry>
-          <box size="${gripper_width} ${gripper_height} ${gripper_height}"/>
-        </geometry> -->
       </collision>
       <inertial>
@@ -349,21 +363,28 @@
     <material>Gazebo/DarkGrey</material>
     <turnGravityOff>true</turnGravityOff>
-    <!-- <self_collide>1</self_collide> -->
+    <self_collide>1</self_collide>
   </gazebo>
   <gazebo reference="upper_base">
-    <turnGravityOff>true</turnGravityOff>
+    <material>Gazebo/LightGrey</material>
+    <turnGravityOff>true</turnGravityOff>
+    <self_collide>1</self_collide>
   </gazebo>
   <gazebo reference="upper_arm">
-    <turnGravityOff>true</turnGravityOff>
     <material>Gazebo/DarkGrey</material>
+    <turnGravityOff>true</turnGravityOff>
+    <self_collide>1</self_collide>
   </gazebo>
   <gazebo reference="lower_arm">
-    <turnGravityOff>true</turnGravityOff>
+    <material>Gazebo/LightGrey</material>
+    <turnGravityOff>true</turnGravityOff>
+    <self_collide>1</self_collide>
   </gazebo>
   <gazebo reference="wrist">
     <turnGravityOff>true</turnGravityOff>
     <material>Gazebo/DarkGrey</material>
+    <self_collide>1</self_collide>
   </gazebo>
   <gazebo reference="gripper_base">
+    <material>Gazebo/LightGrey</material>
     <turnGravityOff>true</turnGravityOff>
   </gazebo>

Commit message: joint naming error and PID parameters

File: al5d_description/urdf/al5d_cad.xacro (robot description, xacro)
@@ -280,5 +280,5 @@
     </link>
     <!-- joints -->
-    <joint name="base" type="fixed">
+    <joint name="base_joint" type="fixed">
       <origin xyz="0 0 0" rpy="0 0 0"/>
       <parent link="world"/>

Commit message: Working collision sensors for all bodies

File: al5d_description/urdf/al5d_cad.xacro (robot description, xacro)
@@ -248,11 +248,5 @@
       </inertial>
     </link>
-    <link name="end">
-      <!-- <visual>
-        <geometry>
-          <sphere radius=".001" />
-        </geometry>
-      </visual> -->
-    </link>
+    <link name="end"></link>
     <link name="xaxis">
       <visual>
@@ -362,24 +356,24 @@
   <gazebo reference="base">
     <material>Gazebo/DarkGrey</material>
-    <turnGravityOff>true</turnGravityOff>
+    <!-- <turnGravityOff>true</turnGravityOff> -->
     <self_collide>1</self_collide>
   </gazebo>
   <gazebo reference="upper_base">
     <material>Gazebo/LightGrey</material>
-    <turnGravityOff>true</turnGravityOff>
+    <!-- <turnGravityOff>true</turnGravityOff> -->
     <self_collide>1</self_collide>
   </gazebo>
   <gazebo reference="upper_arm">
     <material>Gazebo/DarkGrey</material>
-    <turnGravityOff>true</turnGravityOff>
+    <!-- <turnGravityOff>true</turnGravityOff> -->
     <self_collide>1</self_collide>
   </gazebo>
   <gazebo reference="lower_arm">
     <material>Gazebo/LightGrey</material>
-    <turnGravityOff>true</turnGravityOff>
+    <!-- <turnGravityOff>true</turnGravityOff> -->
     <self_collide>1</self_collide>
   </gazebo>
   <gazebo reference="wrist">
-    <turnGravityOff>true</turnGravityOff>
+    <!-- <turnGravityOff>true</turnGravityOff> -->
     <material>Gazebo/DarkGrey</material>
     <self_collide>1</self_collide>
@@ -387,30 +381,79 @@
   <gazebo reference="gripper_base">
     <material>Gazebo/LightGrey</material>
-    <turnGravityOff>true</turnGravityOff>
+    <!-- <turnGravityOff>true</turnGravityOff> -->
   </gazebo>
   <gazebo reference="gripper_leftfinger">
-    <turnGravityOff>true</turnGravityOff>
+    <!-- <turnGravityOff>true</turnGravityOff> -->
     <material>Gazebo/DarkGrey</material>
     <self_collide>1</self_collide>
   </gazebo>
   <gazebo reference="gripper_rightfinger">
-    <turnGravityOff>true</turnGravityOff>
+    <!-- <turnGravityOff>true</turnGravityOff> -->
     <material>Gazebo/DarkGrey</material>
     <self_collide>1</self_collide>
   </gazebo>
   <gazebo reference="end">
-    <turnGravityOff>true</turnGravityOff>
+    <!-- <turnGravityOff>true</turnGravityOff> -->
   </gazebo>
   <gazebo reference="xaxis">
     <material>Gazebo/RedTransparentOverlay</material>
-    <turnGravityOff>true</turnGravityOff>
+    <!-- <turnGravityOff>true</turnGravityOff> -->
   </gazebo>
   <gazebo reference="yaxis">
     <material>Gazebo/GreenTransparentOverlay</material>
-    <turnGravityOff>true</turnGravityOff>
+    <!-- <turnGravityOff>true</turnGravityOff> -->
   </gazebo>
   <gazebo reference="zaxis">
     <material>Gazebo/BlueTransparentOverlay</material>
-    <turnGravityOff>true</turnGravityOff>
-  </gazebo>
+    <!-- <turnGravityOff>true</turnGravityOff> -->
+  </gazebo>
+<!-- WORKING BASE -->
+  <!-- <gazebo reference="base">
+    <sensor type="contact" name="your_link_contact_sensor">
+      <update_rate>50.0</update_rate>
+      <always_on>1</always_on>
+      <contact>
+        <collision>base_collision_collision</collision>
+      </contact>
+      <plugin name="gazebo_ros_bumper_controller" filename="libgazebo_ros_bumper.so">
+        <alwaysOn>true</alwaysOn>
+        <updateRate>50.0</updateRate>
+        <bumperTopicName>/base/collision</bumperTopicName>
+        <frameName>base</frameName>
+      </plugin>
+    </sensor>
+  </gazebo> -->
+  <!-- <gazebo reference="lower_arm">
+    <sensor type="contact" name="lower_arm_contact">
+      <update_rate>10.0</update_rate>
+      <always_on>1</always_on>
+      <contact>
+        <collision>lower_arm_collision_collision</collision>
+        <collision>servo_collision_collision</collision>
+      </contact>
+      <plugin name="gazebo_ros_bumper_controller" filename="libgazebo_ros_bumper.so">
+        <alwaysOn>true</alwaysOn>
+        <updateRate>50.0</updateRate>
+        <bumperTopicName>/collision/lower_arm</bumperTopicName>
+        <frameName>lower_arm</frameName>
+      </plugin>
+    </sensor>
+  </gazebo> -->
+  <xacro:include filename="touch.xacro" />
+  <xacro:touch frame="base" collision_geometry="base_collision"/>
+  <xacro:touch frame="upper_base" collision_geometry="upper_base_collision"/>
+  <xacro:touch frame="upper_base" collision_geometry="upper_base_collision_1"/>
+  <xacro:touch frame="upper_arm" collision_geometry="upper_arm_collision"/>
+  <xacro:touch frame="upper_arm" collision_geometry="upper_arm_collision_1"/>
+  <xacro:touch frame="upper_arm" collision_geometry="upper_arm_collision_2"/>
+  <xacro:touch frame="lower_arm" collision_geometry="lower_arm_collision"/>
+  <xacro:touch frame="lower_arm" collision_geometry="lower_arm_collision_1"/>
+  <xacro:touch frame="lower_arm" collision_geometry="lower_arm_collision_2"/>
+  <xacro:touch frame="wrist" collision_geometry="wrist_collision"/>
+  <xacro:touch frame="wrist" collision_geometry="wrist_collision_1"/>
+  <xacro:touch frame="wrist" collision_geometry="wrist_collision_2"/>
+  <xacro:touch frame="gripper_base" collision_geometry="gripper_base_collision"/>
+  <xacro:touch frame="gripper_base" collision_geometry="gripper_base_collision_1"/>
+  <xacro:touch frame="gripper_leftfinger" collision_geometry="gripper_leftfinger_collision"/>
+  <xacro:touch frame="gripper_rightfinger" collision_geometry="gripper_rightfinger_collision"/>
 </robot>

Commit message: Working collision flag

File: al5d_description/urdf/al5d_cad.xacro (robot description, xacro)
@@ -356,24 +356,19 @@
   <gazebo reference="base">
     <material>Gazebo/DarkGrey</material>
-    <!-- <turnGravityOff>true</turnGravityOff> -->
     <self_collide>1</self_collide>
   </gazebo>
   <gazebo reference="upper_base">
     <material>Gazebo/LightGrey</material>
-    <!-- <turnGravityOff>true</turnGravityOff> -->
     <self_collide>1</self_collide>
   </gazebo>
   <gazebo reference="upper_arm">
     <material>Gazebo/DarkGrey</material>
-    <!-- <turnGravityOff>true</turnGravityOff> -->
     <self_collide>1</self_collide>
   </gazebo>
   <gazebo reference="lower_arm">
     <material>Gazebo/LightGrey</material>
-    <!-- <turnGravityOff>true</turnGravityOff> -->
     <self_collide>1</self_collide>
   </gazebo>
   <gazebo reference="wrist">
-    <!-- <turnGravityOff>true</turnGravityOff> -->
     <material>Gazebo/DarkGrey</material>
     <self_collide>1</self_collide>
@@ -381,63 +376,28 @@
   <gazebo reference="gripper_base">
     <material>Gazebo/LightGrey</material>
-    <!-- <turnGravityOff>true</turnGravityOff> -->
   </gazebo>
   <gazebo reference="gripper_leftfinger">
-    <!-- <turnGravityOff>true</turnGravityOff> -->
     <material>Gazebo/DarkGrey</material>
     <self_collide>1</self_collide>
   </gazebo>
   <gazebo reference="gripper_rightfinger">
-    <!-- <turnGravityOff>true</turnGravityOff> -->
     <material>Gazebo/DarkGrey</material>
     <self_collide>1</self_collide>
   </gazebo>
   <gazebo reference="end">
-    <!-- <turnGravityOff>true</turnGravityOff> -->
   </gazebo>
   <gazebo reference="xaxis">
     <material>Gazebo/RedTransparentOverlay</material>
-    <!-- <turnGravityOff>true</turnGravityOff> -->
   </gazebo>
   <gazebo reference="yaxis">
     <material>Gazebo/GreenTransparentOverlay</material>
-    <!-- <turnGravityOff>true</turnGravityOff> -->
   </gazebo>
   <gazebo reference="zaxis">
     <material>Gazebo/BlueTransparentOverlay</material>
-    <!-- <turnGravityOff>true</turnGravityOff> -->
-  </gazebo>
-<!-- WORKING BASE -->
-  <!-- <gazebo reference="base">
-    <sensor type="contact" name="your_link_contact_sensor">
-      <update_rate>50.0</update_rate>
-      <always_on>1</always_on>
-      <contact>
-        <collision>base_collision_collision</collision>
-      </contact>
-      <plugin name="gazebo_ros_bumper_controller" filename="libgazebo_ros_bumper.so">
-        <alwaysOn>true</alwaysOn>
-        <updateRate>50.0</updateRate>
-        <bumperTopicName>/base/collision</bumperTopicName>
-        <frameName>base</frameName>
-      </plugin>
-    </sensor>
-  </gazebo> -->
-  <!-- <gazebo reference="lower_arm">
-    <sensor type="contact" name="lower_arm_contact">
-      <update_rate>10.0</update_rate>
-      <always_on>1</always_on>
-      <contact>
-        <collision>lower_arm_collision_collision</collision>
-        <collision>servo_collision_collision</collision>
-      </contact>
-      <plugin name="gazebo_ros_bumper_controller" filename="libgazebo_ros_bumper.so">
-        <alwaysOn>true</alwaysOn>
-        <updateRate>50.0</updateRate>
-        <bumperTopicName>/collision/lower_arm</bumperTopicName>
-        <frameName>lower_arm</frameName>
-      </plugin>
-    </sensor>
-  </gazebo> -->
+  </gazebo>
+  <!-- TO GET NAMES OF COLLISION: -->
+  <!-- rosrun xacro xacro al5d_cad.xacro > temp.urdf -->
+  <!-- gz sdf -p temp.urdf > temp.sdf -->
+  <!-- Check names in temp.sdf -->
   <xacro:include filename="touch.xacro" />
   <xacro:touch frame="base" collision_geometry="base_collision"/>
