Commit message: Now there are two of them

File: al5d_description/urdf/al5d_cad.xacro (robot description, xacro)
@@ -20,4 +20,5 @@
     <xacro:property name="axis_length" value="0.03" />
     <xacro:property name="axis_width" value="0.001" />
+    <xacro:arg name="color" default="black" />
     <xacro:property name="inertia_block">
       <inertial>
@@ -371,6 +372,21 @@
   </gazebo>
   <xacro:include filename="touch.xacro" />
+  <xacro:macro name="colorize">
+    <visual>
+      <material>
+        <ambient>$(arg color)</ambient>
+        <diffuse>$(arg color)</diffuse>
+        <specular>$(arg color)</specular>
+        <emissive>0 0 0 0</emissive>
+      </material>
+    </visual>
+  </xacro:macro>
+<!-- 0.7137254 0.3254902 0.2352941 1 -->
+ <!-- TO GET NAMES OF COLLISION GEOMETRY: -->
+ <!-- rosrun xacro xacro al5d_cad.xacro > temp.urdf -->
+ <!-- gz sdf -p temp.urdf > temp.sdf -->
+ <!-- Check names in temp.sdf -->
   <gazebo reference="base">
-    <material>Gazebo/DarkGrey</material>
+    <xacro:colorize />
     <self_collide>1</self_collide>
     <xacro:touch frame="base" collision_geometry="base_collision"/>
@@ -383,5 +399,5 @@
   </gazebo>
   <gazebo reference="upper_arm">
-    <material>Gazebo/DarkGrey</material>
+    <xacro:colorize />
     <self_collide>1</self_collide>
     <xacro:touch frame="upper_arm" collision_geometry="upper_arm_collision"/>
@@ -397,5 +413,5 @@
   </gazebo>
   <gazebo reference="wrist">
-    <material>Gazebo/DarkGrey</material>
+    <xacro:colorize />
     <self_collide>1</self_collide>
     <xacro:touch frame="wrist" collision_geometry="wrist_collision"/>
@@ -409,5 +425,5 @@
   </gazebo>
   <gazebo reference="gripper_leftfinger">
-    <material>Gazebo/DarkGrey</material>
+    <xacro:colorize />
     <self_collide>1</self_collide>
     <turnGravityOff>true</turnGravityOff>
@@ -415,5 +431,5 @@
   </gazebo>
   <gazebo reference="gripper_rightfinger">
-    <material>Gazebo/DarkGrey</material>
+    <xacro:colorize />
     <self_collide>1</self_collide>
     <turnGravityOff>true</turnGravityOff>
@@ -431,24 +447,3 @@
     <material>Gazebo/BlueTransparentOverlay</material>
   </gazebo>
-  <!-- TO GET NAMES OF COLLISION: -->
-  <!-- rosrun xacro xacro al5d_cad.xacro > temp.urdf -->
-  <!-- gz sdf -p temp.urdf > temp.sdf -->
-  <!-- Check names in temp.sdf -->
-  <!-- <xacro:include filename="touch.xacro" />
-  <xacro:touch frame="base" collision_geometry="base_collision"/>
-  <xacro:touch frame="upper_base" collision_geometry="upper_base_collision"/>
-  <xacro:touch frame="upper_base" collision_geometry="upper_base_collision_1"/>
-  <xacro:touch frame="upper_arm" collision_geometry="upper_arm_collision"/>
-  <xacro:touch frame="upper_arm" collision_geometry="upper_arm_collision_1"/>
-  <xacro:touch frame="upper_arm" collision_geometry="upper_arm_collision_2"/>
-  <xacro:touch frame="lower_arm" collision_geometry="lower_arm_collision"/>
-  <xacro:touch frame="lower_arm" collision_geometry="lower_arm_collision_1"/>
-  <xacro:touch frame="lower_arm" collision_geometry="lower_arm_collision_2"/>
-  <xacro:touch frame="wrist" collision_geometry="wrist_collision"/>
-  <xacro:touch frame="wrist" collision_geometry="wrist_collision_1"/>
-  <xacro:touch frame="wrist" collision_geometry="wrist_collision_2"/>
-  <xacro:touch frame="gripper_base" collision_geometry="gripper_base_collision"/>
-  <xacro:touch frame="gripper_base" collision_geometry="gripper_base_collision_1"/>
-  <xacro:touch frame="gripper_leftfinger" collision_geometry="gripper_leftfinger_collision"/>
-  <xacro:touch frame="gripper_rightfinger" collision_geometry="gripper_rightfinger_collision"/> -->
 </robot>

Commit message: Retuning PID and effort limits

File: al5d_description/urdf/al5d_cad.xacro (robot description, xacro)
@@ -301,5 +301,5 @@
       <child link="upper_base"/>
       <axis xyz="0 0 1"/>
-      <limit lower="-1.4" upper="1.4" effort="10" velocity="3.67"/>
+      <limit lower="-1.4" upper="1.4" effort=".5" velocity="3.67"/>
     </joint>
     <joint name="shoulder_tilt" type="revolute">
@@ -308,5 +308,5 @@
       <child link="upper_arm"/>
       <axis xyz="0 0 -1"/>
-      <limit lower="-1.2" upper="1.4" effort="10" velocity="3.32"/>
+      <limit lower="-1.2" upper="1.4" effort="3" velocity="3.32"/>
     </joint>
     <joint name="elbow_tilt" type="revolute">
@@ -315,5 +315,5 @@
       <child link="lower_arm"/>
       <axis xyz="0 0 -1"/>
-      <limit lower="-1.8" upper="1.7" effort="10" velocity="3.67"/>
+      <limit lower="-1.8" upper="1.7" effort="4" velocity="3.67"/>
     </joint>
     <joint name="wrist_tilt" type="revolute">
@@ -322,5 +322,5 @@
       <child link="wrist"/>
       <axis xyz="0 0 -1"/>
-      <limit lower="-1.9" upper="1.7" effort="10" velocity="6.98"/>
+      <limit lower="-1.9" upper="1.7" effort="1" velocity="6.98"/>
     </joint>
     <joint name="wrist_rotate" type="revolute">
@@ -329,5 +329,5 @@
       <child link="gripper_base"/>
       <axis xyz="1 0 0"/>
-      <limit lower="-2" upper="1.5" effort="10" velocity="6.98"/>
+      <limit lower="-2" upper="1.5" effort="1" velocity="6.98"/>
     </joint>
     <joint name="open_gripperright" type="prismatic">

Commit message: Adding lynx.command(...)

File: al5d_description/urdf/al5d_cad.xacro (robot description, xacro)
@@ -315,5 +315,5 @@
       <child link="lower_arm"/>
       <axis xyz="0 0 -1"/>
-      <limit lower="-1.8" upper="1.7" effort="4" velocity="3.67"/>
+      <limit lower="-1.8" upper="1.7" effort="2" velocity="3.67"/>
     </joint>
     <joint name="wrist_tilt" type="revolute">

Commit message: reverting PID gains and effort limits

File: al5d_description/urdf/al5d_cad.xacro (robot description, xacro)
@@ -301,5 +301,5 @@
       <child link="upper_base"/>
       <axis xyz="0 0 1"/>
-      <limit lower="-1.4" upper="1.4" effort=".5" velocity="3.67"/>
+      <limit lower="-1.4" upper="1.4" effort="10" velocity="3.67"/>
     </joint>
     <joint name="shoulder_tilt" type="revolute">
@@ -308,5 +308,5 @@
       <child link="upper_arm"/>
       <axis xyz="0 0 -1"/>
-      <limit lower="-1.2" upper="1.4" effort="3" velocity="3.32"/>
+      <limit lower="-1.2" upper="1.4" effort="10" velocity="3.32"/>
     </joint>
     <joint name="elbow_tilt" type="revolute">
@@ -315,5 +315,5 @@
       <child link="lower_arm"/>
       <axis xyz="0 0 -1"/>
-      <limit lower="-1.8" upper="1.7" effort="2" velocity="3.67"/>
+      <limit lower="-1.8" upper="1.7" effort="10" velocity="3.67"/>
     </joint>
     <joint name="wrist_tilt" type="revolute">
@@ -322,5 +322,5 @@
       <child link="wrist"/>
       <axis xyz="0 0 -1"/>
-      <limit lower="-1.9" upper="1.7" effort="1" velocity="6.98"/>
+      <limit lower="-1.9" upper="1.7" effort="10" velocity="6.98"/>
     </joint>
     <joint name="wrist_rotate" type="revolute">
@@ -329,5 +329,5 @@
       <child link="gripper_base"/>
       <axis xyz="1 0 0"/>
-      <limit lower="-2" upper="1.5" effort="1" velocity="6.98"/>
+      <limit lower="-2" upper="1.5" effort="10" velocity="6.98"/>
     </joint>
     <joint name="open_gripperright" type="prismatic">
